Commit message: 안정적인 기립, 안정화된 물리법칙

File: src/quadruped_description/urdf/quadruped.urdf.xacro (robot description, xacro)
@@ -1,31 +1,47 @@
 <?xml version="1.0"?>
-<robot name="quadruped" xmlns:xacro="http://www.ros.org/wiki/xacro">
+<robot xmlns:xacro="http://www.ros.org/wiki/xacro" name="quadruped">
   <material name="blue"><color rgba="0 0 0.8 1"/></material>
   <material name="black"><color rgba="0.1 0.1 0.1 1"/></material>
+  <material name="yellow"><color rgba="0.9 0.8 0.0 1"/></material>
   <xacro:property name="PI" value="3.1415926535"/>
   <link name="base_footprint"/>
   <joint name="base_joint" type="fixed"><parent link="base_footprint"/><child link="base_link"/><origin xyz="0 0 0"/></joint>
   <link name="base_link">
-    <visual><origin xyz="0 0 0.05"/><geometry><box size="0.2 0.12 0.05"/></geometry><material name="blue"/></visual>
-    <collision><origin xyz="0 0 0.05"/><geometry><box size="0.2 0.12 0.05"/></geometry></collision>
-    <inertial><origin xyz="0 0 0.05"/><mass value="2.0"/><inertia ixx="0.01" ixy="0" ixz="0" iyy="0.01" iyz="0" izz="0.01"/></inertial>
-  </link>
+  <visual><origin xyz="0 0 0.1"/><geometry><box size="0.4 0.24 0.1"/></geometry><material name="blue"/></visual>
+  <collision><origin xyz="0 0 0.1"/><geometry><box size="0.4 0.24 0.1"/></geometry></collision>
+  <inertial>
+    <origin xyz="0.08 0 0.1"/>
+    <mass value="4.0"/>
+    <inertia ixx="0.0229" iyy="0.0567" izz="0.0731" ixy="0" ixz="0" iyz="0"/>
+  </inertial>
+</link>
   <xacro:macro name="simple_leg" params="pos x y reflect">
-    <joint name="${pos}_shoulder_joint" type="revolute"><parent link="base_link"/><child link="${pos}_shoulder_link"/><origin xyz="${x} ${y} 0.05"/><axis xyz="1 0 0"/><limit effort="100.0" lower="-0.78" upper="0.78" velocity="1.0"/></joint>
-    <link name="${pos}_shoulder_link"><visual><origin rpy="${PI/2} 0 0" xyz="0 ${reflect*0.02} 0"/><geometry><cylinder radius="0.02" length="0.04"/></geometry><material name="black"/></visual><inertial><mass value="0.2"/><inertia ixx="0.001" ixy="0" ixz="0" iyy="0.001" iyz="0" izz="0.001"/></inertial></link>
-    <joint name="${pos}_leg_joint" type="revolute"><parent link="${pos}_shoulder_link"/><child link="${pos}_leg_link"/><origin xyz="0 ${reflect*0.04} 0"/><axis xyz="0 1 0"/><limit effort="100.0" lower="-2.6" upper="2.6" velocity="1.0"/></joint>
-    <link name="${pos}_leg_link"><visual><origin xyz="0 0 -0.05"/><geometry><box size="0.02 0.02 0.1"/></geometry><material name="blue"/></visual><collision><origin xyz="0 0 -0.05"/><geometry><box size="0.02 0.02 0.1"/></geometry></collision><inertial><origin xyz="0 0 -0.05"/><mass value="0.2"/><inertia ixx="0.001" ixy="0" ixz="0" iyy="0.001" iyz="0" izz="0.001"/></inertial></link>
-    <joint name="${pos}_foot_joint" type="revolute"><parent link="${pos}_leg_link"/><child link="${pos}_foot_link"/><origin xyz="0 0 -0.1"/><axis xyz="0 1 0"/><limit effort="100.0" lower="-2.6" upper="2.6" velocity="1.0"/></joint>
-    <link name="${pos}_foot_link"><visual><origin xyz="0 0 -0.05"/><geometry><box size="0.015 0.015 0.1"/></geometry><material name="black"/></visual><collision><origin xyz="0 0 -0.05"/><geometry><box size="0.015 0.015 0.1"/></geometry></collision><inertial><origin xyz="0 0 -0.05"/><mass value="0.2"/><inertia ixx="0.001" ixy="0" ixz="0" iyy="0.001" iyz="0" izz="0.001"/></inertial></link>
-    <link name="${pos}_toe_link"><visual><geometry><sphere radius="0.015"/></geometry><material name="black"/></visual><collision><geometry><sphere radius="0.015"/></geometry></collision><inertial><mass value="0.1"/><inertia ixx="0.0001" ixy="0" ixz="0" iyy="0.0001" iyz="0" izz="0.0001"/></inertial></link>
-    <joint name="${pos}_toe_joint" type="fixed"><parent link="${pos}_foot_link"/><child link="${pos}_toe_link"/><origin xyz="0 0 -0.1"/></joint>
-    <gazebo reference="${pos}_toe_link"><mu1>100.0</mu1><mu2>100.0</mu2><kp>1000000.0</kp><kd>100.0</kd></gazebo>
+    <joint name="${pos}_shoulder_joint" type="revolute"><parent link="base_link"/><child link="${pos}_shoulder_link"/><axis xyz="1 0 0"/><origin xyz="${x} ${y} 0.1"/><limit effort="1000.0" lower="-3.14" upper="3.14" velocity="2.0"/><dynamics damping="0.1" friction="0.05"/></joint>
+    <link name="${pos}_shoulder_link"><visual><origin rpy="${PI/2} 0 0" xyz="0 ${reflect*0.04} 0"/><geometry><cylinder radius="0.04" length="0.08"/></geometry><material name="black"/></visual><inertial><mass value="0.4"/><inertia ixx="0.0229" iyy="0.0567" izz="0.0731" ixy="0" ixz="0" iyz="0"/></inertial></link>
+    <joint name="${pos}_leg_joint" type="revolute"><parent link="${pos}_shoulder_link"/><child link="${pos}_leg_link"/><axis xyz="0 1 0"/><origin xyz="0 ${reflect*0.08} 0"/><limit effort="1000.0" lower="-2.6" upper="2.6" velocity="2.0"/><dynamics damping="0.1" friction="0.05"/></joint>
+    <link name="${pos}_leg_link"><visual><origin xyz="0 0 -0.1"/><geometry><box size="0.04 0.04 0.2"/></geometry><material name="yellow"/></visual><collision><origin xyz="0 0 -0.1"/><geometry><box size="0.04 0.04 0.2"/></geometry></collision><inertial><origin xyz="0 0 -0.1"/><mass value="0.4"/><inertia ixx="0.00139" iyy="0.00139" izz="0.00011" ixy="0" ixz="0" iyz="0"/></inertial></link>
+    <joint name="${pos}_foot_joint" type="revolute"><parent link="${pos}_leg_link"/><child link="${pos}_foot_link"/><axis xyz="0 1 0"/><origin xyz="0 0 -0.2"/><limit effort="1000.0" lower="-2.6" upper="2.6" velocity="2.0"/><dynamics damping="0.1" friction="0.05"/></joint>
+    <link name="${pos}_foot_link"><visual><origin xyz="0 0 -0.1"/><geometry><box size="0.03 0.03 0.2"/></geometry><material name="black"/></visual><collision><origin xyz="0 0 -0.1"/><geometry><box size="0.03 0.03 0.2"/></geometry></collision><inertial><origin xyz="0 0 -0.1"/><mass value="0.4"/><inertia ixx="0.00135" iyy="0.00135" izz="0.00006" ixy="0" ixz="0" iyz="0"/></inertial></link>
+    <link name="${pos}_toe_link"><visual><geometry><sphere radius="0.03"/></geometry><material name="black"/></visual><collision><geometry><sphere radius="0.03"/></geometry></collision><inertial><mass value="0.2"/><inertia ixx="0.01" iyy="0.01" izz="0.01" ixy="0" ixz="0" iyz="0"/></inertial></link>
+    <joint name="${pos}_toe_joint" type="fixed"><parent link="${pos}_foot_link"/><child link="${pos}_toe_link"/><origin xyz="0.01 0 -0.2"/></joint>
+    <gazebo reference="${pos}_toe_link"><kp>1000000</kp>
+<kd>80</kd>
+<maxVel>1.0</maxVel>
+<minDepth>0.003</minDepth>
+<mu1>2.0</mu1>
+<mu2>2.0</mu2></gazebo>
   </xacro:macro>
-  <xacro:simple_leg pos="front_left" x="0.1" y="0.06" reflect="1"/>
-  <xacro:simple_leg pos="front_right" x="0.1" y="-0.06" reflect="-1"/>
-  <xacro:simple_leg pos="rear_left" x="-0.1" y="0.06" reflect="1"/>
-  <xacro:simple_leg pos="rear_right" x="-0.1" y="-0.06" reflect="-1"/>
+  <xacro:simple_leg pos="front_left"  x="0.2"  y="0.12"  reflect="1"/>
+  <xacro:simple_leg pos="front_right" x="0.2"  y="-0.12" reflect="-1"/>
+  <xacro:simple_leg pos="rear_left"   x="-0.2" y="0.12"  reflect="1"/>
+  <xacro:simple_leg pos="rear_right"  x="-0.2" y="-0.12" reflect="-1"/>
   <ros2_control name="GazeboSystem" type="system"><hardware><plugin>gazebo_ros2_control/GazeboSystem</plugin></hardware>
-    <xacro:macro name="ji" params="name"><joint name="${name}"><command_interface name="position"/><state_interface name="position"/><state_interface name="velocity"/></joint></xacro:macro>
+    <xacro:macro name="ji" params="name">
+    <joint name="${name}">
+      <command_interface name="effort"/>  <!-- position → effort 변경 -->
+      <state_interface name="position"/>
+      <state_interface name="velocity"/>
+    </joint>
+  </xacro:macro>
     <xacro:ji name="front_left_shoulder_joint"/><xacro:ji name="front_left_leg_joint"/><xacro:ji name="front_left_foot_joint"/>
     <xacro:ji name="front_right_shoulder_joint"/><xacro:ji name="front_right_leg_joint"/><xacro:ji name="front_right_foot_joint"/>
